Commit message: added komodo_2 description

File: mobilican_description/komodo_2/urdf/komodo2_gazebo.xacro (robot description, xacro)
@@ -1,5 +1,5 @@
 <?xml version="1.0"?>
-<robot xmlns:xacro="http://www.ros.org/wiki/xacro" name="lizi" description="Lizi robot">
-    <xacro:include filename="$(find mobilican_description)/lizi_2/urdf/lizi.xacro" />
+<robot xmlns:xacro="http://www.ros.org/wiki/xacro" name="Komodo2" description="Komodo robot">
+    <xacro:include filename="$(find mobilican_description)/komodo_2/urdf/komodo2.xacro" />
     <xacro:include filename="$(find mobilican_gazebo)/macros/depth_cam.xacro" />
     <xacro:include filename="$(find mobilican_gazebo)/macros/cam.xacro" />
@@ -15,18 +15,24 @@
     <xacro:arg name="gps" default="false"/>
     <xacro:arg name="lidar" default="false"/>
-    <xacro:arg name="cam" default="false"/>
+    <xacro:arg name="rgb_cam" default="false"/>
     <xacro:arg name="depth_cam" default="false"/>
-   <xacro:if value="$(arg cam)">
-        <xacro:Camera name="rgb_cam"
-                      link="rgb_cam_link"
-                      image_width="1280"
-                      image_height="720"
-                      image_format="R8G8B8"
-                      clip_near="0.02"
-                      clip_far="200"
-                      image_topic="image_raw"
-                      info_topic="info"
-                      update_rate="30"
-                      horizontal_fov="1.064" />
+    <!-- cameras  -->
+    <xacro:if value="$(arg depth_cam)">
+        <xacro:DepthCam name="camera"
+                        link="rgb_cam_link"
+                        optical_frame="camera_depth_optical_frame"
+                        horizontal_fov="1.592"
+                        img_width="1280"
+                        img_height="800"
+                        img_format="B8G8R8"
+                        clip_near="0.1"
+                        clip_far="200"
+                        update_rate="30.0"
+                        image_topic="color/image_raw"
+                        depth_topic="depth/color/image_raw"
+                        cloud_topic="depth/color/points"
+                        info_topic="color/camera_info"
+                        depth_info_topic="depth/camera_info"
+                        pointcloud_cuttoff="0.2" />
     </xacro:if>
     <xacro:if value="$(arg depth_cam)">
@@ -48,4 +54,5 @@
                         pointcloud_cuttoff="0.2" />
     </xacro:if>
+    <!-- Sonars -->
     <xacro:if value="$(arg urf)">
         <xacro:urf name="left" link="left_urf_link" topic="urf/left" fov="${10.0*M_PI/180.0}" min="0.3" max="5.0" update_rate="10"/>
@@ -53,20 +60,23 @@
         <xacro:urf name="rear" link="rear_urf_link" topic="urf/rear" fov="${10.0*M_PI/180.0}" min="0.3" max="5.0" update_rate="10"/>
     </xacro:if>
+    <!-- hokuyo -->
     <xacro:if value="$(arg lidar)">
         <xacro:lidar name="lidar"
-                     link="laser_link"
-                     topic="scan"
-                     update_rate="10"
-                     samples="720"
-                     resolution="1"
-                     min_angle="-1.5707"
-                     max_angle="1.5707"
-                     range_min="0.1"
-                     range_max="30.0"
-                     range_resolution="0.01" />
+                        link="laser_link"
+                        topic="scan"
+                        update_rate="10"
+                        samples="720"
+                        resolution="1"
+                        min_angle="-1.5707"
+                        max_angle="1.5707"
+                        range_min="0.1"
+                        range_max="30.0"
+                        range_resolution="0.01" />
     </xacro:if>
+    <!-- GPS   -->
     <xacro:if value="$(arg gps)">
         <xacro:gps link="base_link" hz="5" topic="gps" lat="31.262218" long="34.80146100" alt="298"/>
     </xacro:if>
+    <!-- IMU   -->
     <xacro:if value="$(arg imu)">
         <xacro:imu link="base_link" hz="50" topic="imu" />
@@ -163,19 +173,4 @@
     </gazebo>
     <gazebo reference="base_link">
-        <material>Gazebo/Grass</material>
-    </gazebo>
-    <gazebo reference="left_urf_link">
-        <material>Gazebo/Black</material>
-    </gazebo>
-    <gazebo reference="rear_urf_link">
-        <material>Gazebo/Black</material>
-    </gazebo>
-    <gazebo reference="right_urf_link">
-        <material>Gazebo/Black</material>
-    </gazebo>
-    <gazebo reference="laser_link">
-        <material>Gazebo/DarkGrey</material>
-    </gazebo>
-    <gazebo reference="camera_link">
         <material>Gazebo/Grey</material>
     </gazebo>
