Commit message: updating installtion

File: mobilican_description/lizi_2/urdf/lizi_gazebo.xacro (robot description, xacro)
@@ -116,6 +116,6 @@
         </transmission>
     </xacro:if>
-    <xacro:property name="mu1" value="1.0" />
-    <xacro:property name="mu2" value="1.0" />
+    <xacro:property name="mu1" value="0.7" />
+    <xacro:property name="mu2" value="0.7" />
     <gazebo reference="front_left_wheel_link">
         <!-- kp and kd for rubber -->
