Commit message: trx fixes

File: mobilican_description/trx/urdf/trx.urdf (robot description, URDF)
Before this commit: robot trx_robot, 14 links, 13 joints
Links:
- link base_link: geometry collision box size=0.505 0.49 0.30; visual mesh filename=package://mobilican_description/trx/meshes/base_link.STL
- link wheel_front_left: geometry collision cylinder length=0.05 radius=0.1016; visual mesh filename=package://mobilican_description/trx/meshes/wheel.STL
- link wheel_front_right: geometry collision cylinder length=0.05 radius=0.1016; visual mesh filename=package://mobilican_description/trx/meshes/wheel.STL

File: mobilican_description/trx/urdf/trx_gazebo.xacro (robot description, xacro)
@@ -1,5 +1,5 @@
 <?xml version="1.0"?>
 <robot xmlns:xacro="http://www.ros.org/wiki/xacro" name="trx_robot" description="trx robot">
-    <xacro:include filename="$(find trx_description)/urdf/trx.urdf" />
+    <xacro:include filename="$(find mobilican_description)/trx/urdf/trx.urdf" />
     <xacro:include filename="$(find mobilican_gazebo)/macros/depth_cam.xacro" />
     <xacro:include filename="$(find mobilican_gazebo)/macros/urf.xacro" />
@@ -7,5 +7,5 @@
     <xacro:include filename="$(find mobilican_gazebo)/macros/imu.xacro" />
     <xacro:include filename="$(find mobilican_gazebo)/macros/cam.xacro" />
-    <xacro:include filename="$(find trx_gazebo)/macros/VLP-16.urdf.xacro"/>
+    <xacro:include filename="$(find mobilican_gazebo)/macros/VLP-16.urdf.xacro"/>
     <xacro:property name="M_PI" value="3.14159265358979" />
     <xacro:property name="URF_FOV" value="${10.0*M_PI/180}" />
