Commit message: added pick and place demo + some fixes

File: mobilican_description/armadillo_2/urdf/armadillo2_gazebo.xacro (robot description, xacro)
@@ -92,77 +92,59 @@
         </plugin>
     </gazebo>
-    <gazebo reference="left_finger_link">
-        <kp>1000000.0</kp>
-        <kd>1.0</kd>
-        <mu1>1.0</mu1>
-        <mu2>1.0</mu2>
-        <fdir1>0 0 1</fdir1>
-        <maxVel>1.0</maxVel>
-        <minDepth>0.00</minDepth>
-    </gazebo>
+    <transmission name="left_wheel_joint_trans">
+        <type>transmission_interface/SimpleTransmission</type>
+        <joint name="left_wheel_joint">
+            <hardwareInterface>VelocityJointInterface</hardwareInterface>
+        </joint>
+        <actuator name="left_wheel_joint_motor">
+            <mechanicalReduction>1</mechanicalReduction>
+        </actuator>
+    </transmission>
+    <transmission name="right_wheel_joint_trans">
+        <type>transmission_interface/SimpleTransmission</type>
+        <joint name="right_wheel_joint">
+            <hardwareInterface>VelocityJointInterface</hardwareInterface>
+        </joint>
+        <actuator name="right_wheel_joint_motor">
+            <mechanicalReduction>1</mechanicalReduction>
+        </actuator>
+    </transmission>
+    <transmission name="torso_joint_trans">
+        <type>transmission_interface/SimpleTransmission</type>
+        <joint name="torso_joint">
+            <hardwareInterface>PositionJointInterface</hardwareInterface>
+        </joint>
+        <actuator name="torso_joint_motor">
+            <mechanicalReduction>1</mechanicalReduction>
+        </actuator>
+    </transmission>
+    <transmission name="head_pan_joint_trans">
+        <type>transmission_interface/SimpleTransmission</type>
+        <joint name="head_pan_joint">
+            <hardwareInterface>PositionJointInterface</hardwareInterface>
+        </joint>
+        <actuator name="head_pan_joint_motor">
+            <mechanicalReduction>1</mechanicalReduction>
+        </actuator>
+    </transmission>
+    <transmission name="head_tilt_joint_trans">
+        <type>transmission_interface/SimpleTransmission</type>
+        <joint name="head_tilt_joint">
+            <hardwareInterface>PositionJointInterface</hardwareInterface>
+        </joint>
+        <actuator name="head_tilt_joint_motor">
+            <mechanicalReduction>1</mechanicalReduction>
+        </actuator>
+    </transmission>
+    <xacro:property name="mu1" value="2.0" />
+    <xacro:property name="mu2" value="2.0" />
     <gazebo reference="left_finger_joint">
         <implicitSpringDamper>1</implicitSpringDamper>
         <provideFeedback>1</provideFeedback>
     </gazebo>
-    <gazebo reference="right_finger_link">
-        <kp>1000000.0</kp>
-        <kd>1.0</kd>
-        <mu1>1.0</mu1>
-        <mu2>1.0</mu2>
-        <fdir1>0 0 1</fdir1>
-        <maxVel>1.0</maxVel>
-        <minDepth>0.00</minDepth>
-    </gazebo>
     <gazebo reference="right_finger_joint">
         <implicitSpringDamper>1</implicitSpringDamper>
         <provideFeedback>1</provideFeedback>
     </gazebo>
-    <transmission name="left_wheel_joint_trans">
-        <type>transmission_interface/SimpleTransmission</type>
-        <joint name="left_wheel_joint">
-            <hardwareInterface>VelocityJointInterface</hardwareInterface>
-        </joint>
-        <actuator name="left_wheel_joint_motor">
-            <mechanicalReduction>1</mechanicalReduction>
-        </actuator>
-    </transmission>
-    <transmission name="right_wheel_joint_trans">
-        <type>transmission_interface/SimpleTransmission</type>
-        <joint name="right_wheel_joint">
-            <hardwareInterface>VelocityJointInterface</hardwareInterface>
-        </joint>
-        <actuator name="right_wheel_joint_motor">
-            <mechanicalReduction>1</mechanicalReduction>
-        </actuator>
-    </transmission>
-    <transmission name="torso_joint_trans">
-        <type>transmission_interface/SimpleTransmission</type>
-        <joint name="torso_joint">
-            <hardwareInterface>PositionJointInterface</hardwareInterface>
-        </joint>
-        <actuator name="torso_joint_motor">
-            <mechanicalReduction>1</mechanicalReduction>
-        </actuator>
-    </transmission>
-    <transmission name="head_pan_joint_trans">
-        <type>transmission_interface/SimpleTransmission</type>
-        <joint name="head_pan_joint">
-            <hardwareInterface>PositionJointInterface</hardwareInterface>
-        </joint>
-        <actuator name="head_pan_joint_motor">
-            <mechanicalReduction>1</mechanicalReduction>
-        </actuator>
-    </transmission>
-    <transmission name="head_tilt_joint_trans">
-        <type>transmission_interface/SimpleTransmission</type>
-        <joint name="head_tilt_joint">
-            <hardwareInterface>PositionJointInterface</hardwareInterface>
-        </joint>
-        <actuator name="head_tilt_joint_motor">
-            <mechanicalReduction>1</mechanicalReduction>
-        </actuator>
-    </transmission>
-    <xacro:property name="mu1" value="2.0" />
-    <xacro:property name="mu2" value="2.0" />
     <gazebo reference="left_wheel_link">
         <!-- kp and kd for rubber -->
