Commit message: intel enable

File: mobilican_description/armadillo_2/urdf/intel_d435.urdf (robot description, URDF)
Before this commit: robot intel_d435, 1 links, 0 joints
Links:
- added link camera_depth_frame
- added link camera_depth_optical_frame
- added link camera_fisheye_frame
- added link camera_fisheye_optical_frame
- added link camera_left_ir_frame
- added link camera_left_ir_optical_frame
- added link camera_right_ir_frame
- added link camera_right_ir_optical_frame
Joints:
- added joint camera_depth_joint: type fixed, parent camera_link, child camera_depth_frame, origin xyz=0 -0.0122 0 rpy=0 0 0
- added joint camera_depth_optical_joint: type fixed, parent camera_depth_frame, child camera_depth_optical_frame, origin xyz=0 0 0 rpy=${-M_PI/2} 0 ${-M_PI/2}
- added joint camera_fisheye_joint: type fixed, parent camera_link, child camera_fisheye_frame, origin xyz=0 0.0322 0 rpy=0 0 0
- added joint camera_fisheye_optical_joint: type fixed, parent camera_fisheye_frame, child camera_fisheye_optical_frame, origin xyz=0 0 0 rpy=${-M_PI/2} 0 ${-M_PI/2}
- added joint camera_left_ir_joint: type fixed, parent camera_link, child camera_left_ir_frame, origin xyz=0 -0.0322 0 rpy=0 0 0
- added joint camera_left_ir_optical_joint: type fixed, parent camera_left_ir_frame, child camera_left_ir_optical_frame, origin xyz=0 0 0 rpy=${-M_PI/2} 0 ${-M_PI/2}
- added joint camera_right_ir_joint: type fixed, parent camera_link, child camera_right_ir_frame, origin xyz=0 0.0178 0 rpy=0 0 0
- added joint camera_right_ir_optical_joint: type fixed, parent camera_right_ir_frame, child camera_right_ir_optical_frame, origin xyz=0 0 0 rpy=${-M_PI/2} 0 ${-M_PI/2}
