Commit message: fixed updateConfig deadlock warning

File: mobilican_description/armadillo_2/urdf/armadillo2.xacro (robot description, xacro)
@@ -17,5 +17,5 @@
         rpy="0 0 0" />
        <mass
-        value="70" />
+        value="50" />
         <inertia
           ixx="0.31639"
@@ -63,9 +63,13 @@
       </collision>
       <inertial>
-        <mass value="0.01" />
+        <mass value="0.0001" />
         <origin xyz="0 0 0" />
-        <inertia ixx="0.001" ixy="0.0" ixz="0.0"
-                 iyy="0.001" iyz="0.0"
-                 izz="0.001" />
+        <inertia
+        ixx="0.0069046"
+        ixy="-3.8717E-08"
+        ixz="2.0707E-07"
+        iyy="0.01"
+        iyz="-1.0124E-07"
+        izz="0.0069054" />
       </inertial>
     </link>
@@ -83,9 +87,13 @@
       </collision>
       <inertial>
-        <mass value="0.01" />
+        <mass value="0.0001" />
         <origin xyz="0 0 0" />
-        <inertia ixx="0.001" ixy="0.0" ixz="0.0"
-                 iyy="0.001" iyz="0.0"
-                 izz="0.001" />
+        <inertia
+        ixx="0.0069046"
+        ixy="-3.8717E-08"
+        ixz="2.0707E-07"
+        iyy="0.01"
+        iyz="-1.0124E-07"
+        izz="0.0069054" />
       </inertial>
     </link>
@@ -97,10 +105,10 @@
         rpy="0 0 0" />
     <mass
-        value="1.8524" />
+        value="1.5" />
       <inertia
         ixx="0.0069046"
         ixy="-3.8717E-08"
         ixz="2.0707E-07"
-        iyy="0.013153"
+        iyy="0.01"
         iyz="-1.0124E-07"
         izz="0.0069054" />
@@ -152,10 +160,10 @@
         rpy="0 0 0" />
        <mass
-        value="1.8524" />
+        value="1.5" />
       <inertia
         ixx="0.0069046"
         ixy="-3.8717E-08"
         ixz="-2.0707E-07"
-        iyy="0.013153"
+        iyy="0.01"
         iyz="1.0124E-07"
         izz="0.0069054" />
@@ -202,4 +210,18 @@
  <link
     name="caster_left_link">
+     <inertial>
+      <origin
+        xyz="9.16610941069373E-06 -4.99540929455033E-06 8.06098359126817E-06"
+        rpy="0 0 0" />
+       <mass
+        value="1.1" />
+      <inertia
+        ixx="0.0069046"
+        ixy="-3.8717E-08"
+        ixz="-2.0707E-07"
+        iyy="0.01"
+        iyz="1.0124E-07"
+        izz="0.0069054" />
+    </inertial>
     <visual>
       <origin
@@ -262,4 +284,18 @@
   <link
     name="caster_right_link">
+      <inertial>
+      <origin
+        xyz="9.16610941069373E-06 -4.99540929455033E-06 8.06098359126817E-06"
+        rpy="0 0 0" />
+       <mass
+        value="1.1" />
+      <inertia
+        ixx="0.0069046"
+        ixy="-3.8717E-08"
+        ixz="-2.0707E-07"
+        iyy="0.01"
+        iyz="1.0124E-07"
+        izz="0.0069054" />
+    </inertial>
     <visual>
       <origin
@@ -302,7 +338,7 @@
         ixy="2.4285E-05"
         ixz="-0.0045097"
-        iyy="0.06807"
+        iyy="0.0001"
         iyz="-7.4938E-05"
-        izz="0.072852" />
+        izz="0.00032852" />
     </inertial>
     <visual>
@@ -334,5 +370,5 @@
         rpy="0 0 0" />
       <geometry>
-        <box size="0.09 0.5 0.8"/>
+        <box size="0.09 0.5 0.6"/>
       </geometry>
     </collision>
@@ -355,5 +391,5 @@
       effort="0.001"
       velocity="0.1" />
-<dynamics damping="0.1" friction="0"/>
+<!--<dynamics damping="0.1" friction="0"/>-->
   </joint>
   <link
@@ -414,5 +450,5 @@
       effort="0.5"
       velocity="2" />
-<dynamics damping="0.1" friction="0"/>
+<!--<dynamics damping="0.1" friction="0"/>-->
   </joint>
   <link
@@ -473,5 +509,5 @@
       effort="0.5"
       velocity="2" />
-<dynamics damping="0.1" friction="0"/>
+<!--<dynamics damping="0.1" friction="0"/>-->
   </joint>
   <link
@@ -589,5 +625,5 @@
       upper="1.57"
       velocity="2.0" />
-<dynamics damping="0.1" friction="0"/>
+<!--<dynamics damping="0.1" friction="0"/>-->
   </joint>
   <link
@@ -648,5 +684,5 @@
       upper="1.95"
       velocity="2.0" />
-<dynamics damping="0.1" friction="0"/>
+<!--<dynamics damping="0.1" friction="0"/>-->
   </joint>
   <link
@@ -707,5 +743,5 @@
       upper="2.3522"
       velocity="2.0" />
-<dynamics damping="0.1" friction="0"/>
+<!--<dynamics damping="0.1" friction="0"/>-->
   </joint>
   <link
@@ -766,5 +802,5 @@
       upper="1.57"
       velocity="2.0" />
-<dynamics damping="0.1" friction="0"/>
+<!--<dynamics damping="0.1" friction="0"/>-->
   </joint>
   <link
@@ -825,5 +861,5 @@
       upper="1.57"
       velocity="2.0" />
-<dynamics damping="0.1" friction="0"/>
+<!--<dynamics damping="0.1" friction="0"/>-->
   </joint>
   <link
@@ -884,5 +920,5 @@
       upper="3.14"
       velocity="2.0" />
-<dynamics damping="0.5" friction="0.5"/>
+<!--<dynamics damping="0.5" friction="0.5"/>-->
   </joint>
   <link name="gripper_link"/>
@@ -949,5 +985,5 @@
       upper="1.57"
       velocity="0.1" />
-<dynamics damping="0.5" friction="0.5"/>
+<!--<dynamics damping="0.5" friction="0.5"/>-->
   </joint>
   <link
@@ -1008,5 +1044,5 @@
       upper="1.57"
       velocity="0.1" />
-<dynamics damping="0.5" friction="0.5"/>
+<!--<dynamics damping="0.5" friction="0.5"/>-->
   </joint>
     <joint

Commit message: fixed bugs in pick and place demo

File: mobilican_description/armadillo_2/urdf/armadillo2.xacro (robot description, xacro)
@@ -10,19 +10,18 @@
     <origin xyz="0.00 0.00 ${WHEEL_RADIUS-0.0115}" rpy="0.0 0.0 0.0"/>
   </joint>
-  <link
-    name="base_link">
-    <inertial>
-      <origin
-        xyz="-0.012353 0.000122 0.17716"
+ <link name="base_link">
+    <inertial>
+      <origin
+        xyz=" -0.0456493 0.0002660 0.1875887"
         rpy="0 0 0" />
        <mass
-        value="100" />
+        value="42.08611" />
         <inertia
-          ixx="0.31639"
-          ixy="-9.1727E-05"
-          ixz="-0.093044"
-          iyy="0.017997"
-          iyz="5.3231E-05"
-          izz="0.16693" />
+          ixx="2.8470581"
+          ixy="-0.0025756"
+          ixz="-0.3288866"
+          iyy="2.7606341"
+          iyz="-0.0127145"
+          izz="1.0791602" />
         </inertial>
     <visual>
@@ -73,5 +72,5 @@
         izz="0.0069054" />
       </inertial>
-      <damping>3.0</damping>
+      <damping>1.0</damping>
     </link>
     <joint name="caster_back_right_joint" type="fixed">
@@ -98,5 +97,5 @@
         izz="0.0069054" />
       </inertial>
-      <damping>3.0</damping>
+      <damping>1.0</damping>
     </link>
  <link
@@ -138,5 +137,5 @@
       </geometry>
     </collision>
-    <damping>3.0</damping>
+    <damping>1.0</damping>
   </link>
   <joint
@@ -194,5 +193,5 @@
       </geometry>
     </collision>
-    <damping>3.0</damping>
+    <damping>1.0</damping>
   </link>
   <joint
@@ -989,5 +988,5 @@
       upper="1.57"
       velocity="0.1" />
-<!--<dynamics damping="0.5" friction="0.5"/>-->
+    <dynamics damping="0.1" friction="0.5"/>
   </joint>
   <link
@@ -1048,5 +1047,5 @@
       upper="1.57"
       velocity="0.1" />
-<!--<dynamics damping="0.5" friction="0.5"/>-->
+      <dynamics damping="0.1" friction="0.5"/>
   </joint>
     <joint

File: mobilican_description/armadillo_2/urdf/armadillo2_gazebo.xacro (robot description, xacro)
@@ -79,7 +79,7 @@
             <arm>
                 <arm_name>arm</arm_name>
-                <palm_link> wrist_link  </palm_link>
-                <gripper_link> left_finger_link </gripper_link>
-                <gripper_link> right_finger_link </gripper_link>
+                <palm_link>wrist_link</palm_link>
+                <gripper_link>left_finger_link</gripper_link>
+                <gripper_link>right_finger_link</gripper_link>
             </arm>
             <forces_angle_tolerance>100</forces_angle_tolerance>

Commit message: added new world

File: mobilican_description/armadillo_2/urdf/armadillo2.xacro (robot description, xacro)
@@ -99,5 +99,5 @@
       <damping>1.0</damping>
     </link>
- <link
+<link
     name="left_wheel_link">
     <inertial>

Commit message: gaz link1 tested

File: mobilican_description/armadillo_2/urdf/armadillo2.xacro (robot description, xacro)
@@ -333,5 +333,5 @@
   <inertial>
       <origin
-        xyz="-0.059733 -0.00037419 0.54938"
+        xyz="-0.059654 -0.000364 0.549359"
         rpy="0 0 0" />
      <mass
@@ -394,5 +394,4 @@
       effort="0.001"
       velocity="0.1" />
-<!--<dynamics damping="0.1" friction="0"/>-->
   </joint>
   <link
@@ -453,5 +452,4 @@
       effort="0.5"
       velocity="2" />
-<!--<dynamics damping="0.1" friction="0"/>-->
   </joint>
   <link
@@ -512,5 +510,4 @@
       effort="0.5"
       velocity="2" />
-<!--<dynamics damping="0.1" friction="0"/>-->
   </joint>
   <link
@@ -578,11 +575,11 @@
         rpy="0 0 0" />
       <mass
-        value="0.001" />
+        value="0.08" />
       <inertia
         ixx="0.00055596"
-        ixy="9.2522E-12"
-        ixz="9.2226E-12"
+        ixy="0.0"
+        ixz="0.0"
         iyy="0.00016945"
-        iyz="6.1918E-06"
+        iyz="0.0"
         izz="0.00055286" />
     </inertial>
@@ -628,5 +625,4 @@
       upper="1.57"
       velocity="2.0" />
-<!--<dynamics damping="0.1" friction="0"/>-->
   </joint>
   <link

File: mobilican_description/armadillo_2/urdf/armadillo2_gazebo.xacro (robot description, xacro)
@@ -266,3 +266,51 @@
         </actuator>
     </transmission>
+    <!-- Link1 -->
+  <gazebo reference="rotation1_link">
+    <mu1>0.2</mu1>
+    <mu2>0.2</mu2>
+    <material>Gazebo/Grey</material>
+  </gazebo>
+  <!-- Link2 -->
+  <gazebo reference="shoulder1_link">
+    <mu1>0.2</mu1>
+    <mu2>0.2</mu2>
+    <material>Gazebo/Grey</material>
+  </gazebo>
+  <!-- Link3 -->
+  <gazebo reference="shoulder2_link">
+    <mu1>0.2</mu1>
+    <mu2>0.2</mu2>
+    <material>Gazebo/Grey</material>
+  </gazebo>
+  <!-- Link4 -->
+  <gazebo reference="rotation2_link">
+    <mu1>0.2</mu1>
+    <mu2>0.2</mu2>
+    <material>Gazebo/Grey</material>
+  </gazebo>
+  <!-- Link5 -->
+  <gazebo reference="shoulder3_link">
+    <mu1>0.2</mu1>
+    <mu2>0.2</mu2>
+    <material>Gazebo/Grey</material>
+  </gazebo>
+  <!-- Link6 -->
+  <gazebo reference="wrist_link">
+    <mu1>0.2</mu1>
+    <mu2>0.2</mu2>
+    <material>Gazebo/Grey</material>
+  </gazebo>
+  <!-- End Link -->
+  <gazebo reference="right_finger_link">
+    <mu1>0.2</mu1>
+    <mu2>0.2</mu2>
+    <material>Gazebo/Grey</material>
+  </gazebo>
+  <!-- End Link -->
+  <gazebo reference="left_finger_link">
+    <mu1>0.2</mu1>
+    <mu2>0.2</mu2>
+    <material>Gazebo/Grey</material>
+  </gazebo>
 </robot>

Commit message: fixed bugs in pick and place demo

File: mobilican_description/armadillo_2/urdf/armadillo2.xacro (robot description, xacro)
@@ -72,5 +72,5 @@
         izz="0.0069054" />
       </inertial>
-      <damping>1.0</damping>
+      <damping>0.5</damping>
     </link>
     <joint name="caster_back_right_joint" type="fixed">
@@ -97,5 +97,5 @@
         izz="0.0069054" />
       </inertial>
-      <damping>1.0</damping>
+      <damping>0.5</damping>
     </link>
 <link
@@ -137,5 +137,5 @@
       </geometry>
     </collision>
-    <damping>1.0</damping>
+    <damping>0.5</damping>
   </link>
   <joint
@@ -193,5 +193,5 @@
       </geometry>
     </collision>
-    <damping>1.0</damping>
+    <damping>0.5</damping>
   </link>
   <joint
@@ -336,5 +336,5 @@
         rpy="0 0 0" />
      <mass
-        value="0.1" />
+        value="0.005" />
       <inertia
         ixx="0.09579"
@@ -575,5 +575,5 @@
         rpy="0 0 0" />
       <mass
-        value="0.08" />
+        value="0.008" />
       <inertia
         ixx="0.00055596"
@@ -621,5 +621,5 @@
       xyz="0 0 1" />
        <limit
-      effort="0.01"
+      effort="0.001"
       lower="-1.57"
       upper="1.57"
@@ -633,11 +633,11 @@
         rpy="0 0 0" />
       <mass
-        value="0.001" />
+        value="0.009" />
       <inertia
         ixx="0.0043595"
-        ixy="-3.1405E-06"
+        ixy="0.0"
         ixz="0.00053636"
         iyy="0.0041046"
-        iyz="-5.2275E-05"
+        iyz="0.0"
         izz="0.00081871" />
     </inertial>
@@ -683,5 +683,4 @@
       upper="1.95"
       velocity="2.0" />
-<!--<dynamics damping="0.1" friction="0"/>-->
   </joint>
   <link
@@ -695,8 +694,8 @@
       <inertia
         ixx="0.00093237"
-        ixy="-1.0052E-05"
+        ixy="0.0"
         ixz="0.00048929"
         iyy="0.0012859"
-        iyz="-1.3286E-05"
+        iyz="0.0"
         izz="0.00091329" />
     </inertial>
@@ -742,5 +741,4 @@
       upper="2.3522"
       velocity="2.0" />
-<!--<dynamics damping="0.1" friction="0"/>-->
   </joint>
   <link
@@ -754,8 +752,8 @@
       <inertia
         ixx="0.00014092"
-        ixy="1.0984E-09"
-        ixz="1.6669E-08"
+        ixy="0.0"
+        ixz="0.0"
         iyy="8.0775E-05"
-        iyz="-1.7606E-06"
+        iyz="0.0"
         izz="0.00010647" />
     </inertial>
@@ -801,5 +799,4 @@
       upper="1.57"
       velocity="2.0" />
-<!--<dynamics damping="0.1" friction="0"/>-->
   </joint>
   <link
@@ -810,11 +807,11 @@
         rpy="0 0 0" />
       <mass
-        value="0.001" />
+        value="0.00045" />
       <inertia
         ixx="0.00018198"
-        ixy="2.1351E-13"
-        ixz="-2.3815E-13"
+        ixy="0.0"
+        ixz="0.0"
         iyy="0.00015335"
-        iyz="-5.6341E-06"
+        iyz="0.0"
         izz="7.5641E-05" />
     </inertial>
@@ -860,6 +857,6 @@
       upper="1.57"
       velocity="2.0" />
-<!--<dynamics damping="0.1" friction="0"/>-->
-  </joint>
+    <dynamics damping="0.1"/>
+    </joint>
   <link
     name="wrist_link">
@@ -869,11 +866,11 @@
         rpy="0 0 0" />
       <mass
-        value="0.001" />
+        value="0.00043" />
       <inertia
         ixx="4.4099E-05"
-        ixy="-1.2434E-13"
-        ixz="-1.4422E-13"
+        ixy="0.0"
+        ixz="0.0"
         iyy="9.4421E-05"
-        iyz="3.0209E-06"
+        iyz="0.0"
         izz="0.00010114" />
     </inertial>
@@ -919,5 +916,4 @@
       upper="3.14"
       velocity="2.0" />
-<!--<dynamics damping="0.5" friction="0.5"/>-->
   </joint>
   <link name="gripper_link"/>
@@ -934,11 +930,11 @@
         rpy="0 0 0" />
       <mass
-        value="0.001" />
+        value="0.0003" />
       <inertia
         ixx="1.4683E-05"
-        ixy="-1.0482E-21"
-        ixz="1.8423E-20"
+        ixy="0.0"
+        ixz="0.0"
         iyy="1.7304E-05"
-        iyz="9.2811E-07"
+        iyz="0.0"
         izz="4.5506E-06" />
     </inertial>
@@ -993,11 +989,11 @@
         rpy="0 0 0" />
       <mass
-        value="0.001" />
+        value="0.0003" />
       <inertia
         ixx="1.4683E-05"
-        ixy="2.0869E-20"
-        ixz="-3.5787E-20"
+        ixy="0.0"
+        ixz="0.0"
         iyy="1.7304E-05"
-        iyz="-9.2811E-07"
+        iyz="0.0"
         izz="4.5506E-06" />
     </inertial>

File: mobilican_description/armadillo_2/urdf/armadillo2_gazebo.xacro (robot description, xacro)
@@ -155,5 +155,5 @@
         <fdir1>1 0 0</fdir1>
         <maxVel>1.0</maxVel>
-        <minDepth>0.005</minDepth>
+        <minDepth>0.002</minDepth>
         <material>Gazebo/DarkGrey</material>
     </gazebo>
@@ -166,5 +166,5 @@
         <fdir1>1 0 0</fdir1>
         <maxVel>1.0</maxVel>
-        <minDepth>0.005</minDepth>
+        <minDepth>0.002</minDepth>
         <material>Gazebo/DarkGrey</material>
     </gazebo>
@@ -177,5 +177,5 @@
         <fdir1>1 0 0</fdir1>
         <maxVel>1.0</maxVel>
-        <minDepth>0.002</minDepth>
+        <minDepth>0.001</minDepth>
         <material>Gazebo/DarkGrey</material>
     </gazebo>
@@ -188,5 +188,5 @@
         <fdir1>1 0 0</fdir1>
         <maxVel>1.0</maxVel>
-        <minDepth>0.002</minDepth>
+        <minDepth>0.001</minDepth>
         <material>Gazebo/DarkGrey</material>
     </gazebo>
