Commit message: middle of armadillo model

File: mobilican_description/armadillo_2/urdf/armadillo2.xacro (robot description, xacro)
@@ -1,7 +1,7 @@
 <?xml version="1.0"?>
 <robot xmlns:xacro="http://www.ros.org/wiki/xacro" name="armadillo_robot" description="armadillo robot">
- <xacro:property name="M_PI" value="3.1415926535897931" />
- <xacro:property name="WHEEL_RADIUS" value="0.1016" />
- <xacro:include filename="$(find mobilican_description)/armadillo_2/urdf/intel_d435.urdf"/>
+  <xacro:property name="M_PI" value="3.1415926535897931" />
+  <xacro:property name="WHEEL_RADIUS" value="0.1016" />
+  <!-- <xacro:include filename="$(find mobilican_description)/armadillo_2/urdf/intel_d435.urdf"/>
 <link name="base_footprint"/>
  <joint name="base_footprint_joint" type="fixed">
@@ -9,392 +9,196 @@
     <child link="base_link"/>
     <origin xyz="0.00 0.00 ${WHEEL_RADIUS-0.0115}" rpy="0.0 0.0 0.0"/>
-  </joint>
- <link name="base_link">
-    <inertial>
+  </joint>  -->
+  <!-- <link name="base_link">
+    <inertial>
+      <origin xyz=" -0.0456493 0.0002660 0.1875887" rpy="0 0 0" />
+      <mass value="42.0" />
+      <inertia ixx="2.8470581" ixy="0.0" ixz="0.0" iyy="2.7606341" iyz="0.0" izz="1.0791602" />
+    </inertial>
+    <visual>
+      <origin xyz="0 0 0" rpy="0 0 0" />
+      <geometry>
+        <mesh filename="package://mobilican_description/armadillo_2/mesh/base_link.STL" />
+      </geometry>
+      <material name="">
+        <color rgba="0.79216 0.81961 0.93333 1" />
+      </material>
+    </visual>
+    <collision name='base_collision'>
+      <origin xyz="0 0 0" rpy="0 0 0" />
+      <geometry>
+        <mesh filename="package://mobilican_description/armadillo_2/mesh/base_link.STL" />
+      </geometry>
+    </collision>
+  </link> -->
+  <!-- <link name="left_wheel_link">
+    <inertial>
+      <origin xyz="9.16610941069373E-06 4.59070539915452E-09 8.0609835912647E-06" rpy="0 0 0" />
+      <mass value="1.5" />
+      <inertia ixx="0.0069046" ixy="-3.8717E-08" ixz="2.0707E-07" iyy="0.01" iyz="-1.0124E-07" izz="0.0069054" />
+    </inertial>
+    <visual>
+      <origin xyz="0 0 0" rpy="0 0 0" />
+      <geometry>
+        <mesh filename="package://mobilican_description/armadillo_2/mesh/left_wheel_link.STL" />
+      </geometry>
+      <material name="">
+        <color rgba="0.792156862745098 0.819607843137255 0.933333333333333 1" />
+      </material>
+    </visual>
+    <collision>
+      <origin xyz="0 0 0" rpy="1.57079632679 0 0" />
+      <geometry>
+        <cylinder length="0.05" radius="0.1016"/>
+      </geometry>
+    </collision>
+    <damping>0.5</damping>
+  </link> -->
+  <!-- <joint name="left_wheel_joint" type="continuous">
+    <origin xyz="0.063115 0.16085 0.0115" rpy="0 0 0" />
+    <parent link="base_link" />
+    <child link="left_wheel_link" />
+    <axis xyz="0 1 0" />
+    <limit effort="0.1" velocity="10.0" />
+  </joint> -->
+ <!-- <link name="right_wheel_link">
+    <inertial>
+      <origin xyz="9.16610941069373E-06 -4.99540929455033E-06 8.06098359126817E-06" rpy="0 0 0" />
+       <mass value="1.5" />
+      <inertia ixx="0.0069046" ixy="0.0" ixz="0.0" iyy="0.01" iyz="0.0" izz="0.0069054" />
+    </inertial>
+    <visual>
+      <origin xyz="0 0 0" rpy="0 0 0" />
+      <geometry>
+        <mesh filename="package://mobilican_description/armadillo_2/mesh/right_wheel_link.STL" />
+      </geometry>
+      <material name="">
+        <color rgba="0.792156862745098 0.819607843137255 0.933333333333333 1" />
+      </material>
+    </visual>
+   <collision>
+      <origin xyz="0 0 0" rpy="1.57079632679 0 0" />
+      <geometry>
+      <cylinder length="0.05" radius="0.1016"/>
+      </geometry>
+    </collision>
+    <damping>0.5</damping>
+  </link> -->
+  <!-- <joint name="right_wheel_joint" type="continuous">
+    <origin xyz="0.063115 -0.16085 0.0115" rpy="0 0 0" />
+    <parent link="base_link" />
+    <child link="right_wheel_link" />
+    <axis xyz="0 1 0" />
+    <limit effort="0.1" velocity="10.0" />
+  </joint> -->
+ <!-- <link name="caster_left_link">
+     <inertial>
       <origin
-        xyz=" -0.0456493 0.0002660 0.1875887"
+        xyz="-0.2215584 0.1690000 -0.0478000"
         rpy="0 0 0" />
        <mass
-        value="42.08611" />
-        <inertia
-          ixx="2.8470581"
-          ixy="-0.0025756"
-          ixz="-0.3288866"
-          iyy="2.7606341"
-          iyz="-0.0127145"
-          izz="1.0791602" />
-        </inertial>
-    <visual>
-      <origin
-        xyz="0 0 0"
-        rpy="0 0 0" />
-      <geometry>
-        <mesh
-          filename="package://mobilican_description/armadillo_2/mesh/base_link.STL" />
-      </geometry>
-      <material
-        name="">
-        <color
-          rgba="0.79216 0.81961 0.93333 1" />
-      </material>
-    </visual>
- <collision name='base_collision'>
-       <origin
-        xyz="0 0 0"
-        rpy="0 0 0" />
-      <geometry>
-        <mesh
-          filename="package://mobilican_description/armadillo_2/mesh/base_link.STL" />
-      </geometry>
-          </collision>
-  </link>
-    <joint name="caster_back_left_joint" type="fixed">
-      <parent link="base_link"/>
-      <child link="caster_back_left_link"/>
-      <origin xyz="-0.2 0.24 ${-WHEEL_RADIUS+0.0115+0.05}" rpy="${-M_PI/2} 0 0"/>
-    </joint>
-    <link name="caster_back_left_link">
-      <collision>
-        <geometry>
-          <cylinder length="0.06" radius="0.05"/>
-        </geometry>
-        <origin rpy="0 0 0" xyz="0 0 -0.03"/>
-      </collision>
+        value="0.1" />
+      <inertia
+        ixx="0.0000224"
+        ixy="0.0000001"
+        ixz="0.0000006"
+        iyy="0.0000356"
+        iyz="0.0000001"
+        izz="0.0000211" />
+    </inertial>
+    <visual>
+      <origin xyz="0 0 0" rpy="0 0 0" />
+      <geometry>
+        <mesh filename="package://mobilican_description/armadillo_2/mesh/caster_left_link.STL" />
+      </geometry>
+      <material name="">
+        <color rgba="0.792156862745098 0.819607843137255 0.933333333333333 1" />
+      </material>
+    </visual>
+    <collision>
+      <origin xyz="0 0 0" rpy="1.57079632679 0 0" />
+      <geometry>
+      <cylinder length="0.018" radius="0.025"/>
+      </geometry>
+    </collision>
+  </link> -->
+  <!-- <link name="laser_link" /> -->
+  <!-- <joint name="laser_joint" type="fixed">
+    <origin xyz="0.20337 0 0.143" rpy="0 0 0" />
+    <parent link="base_link" />
+    <child link="laser_link" />
+    <axis xyz="0 0 0" />
+  </joint> -->
+  <!-- <link name="front_urf_link" /> -->
+  <!-- <joint name="front_urf_joint" type="fixed">
+    <origin xyz="0.24229 0.00011161 0.068509" rpy="0 0 0" />
+    <parent link="base_link" />
+    <child link="front_urf_link" />
+    <axis xyz="0 0 0" />
+  </joint> -->
+  <!-- <joint name="caster_left_joint" type="fixed">
+    <origin xyz="-0.221558374889189 0.168999999975415 -0.0596832588142329" rpy="0 0 0" />
+    <parent link="base_link" />
+    <child link="caster_left_link" />
+    <axis xyz="0 0 0" />
+  </joint> -->
+  <!-- <link name="caster_right_link">
       <inertial>
-        <mass value="0.0001" />
-        <origin xyz="0 0 0" />
-        <inertia
-        ixx="0.0069046"
-        ixy="-3.8717E-08"
-        ixz="2.0707E-07"
-        iyy="0.01"
-        iyz="-1.0124E-07"
-        izz="0.0069054" />
-      </inertial>
-      <damping>0.5</damping>
-    </link>
-    <joint name="caster_back_right_joint" type="fixed">
-      <parent link="base_link"/>
-      <child link="caster_back_right_link"/>
-      <origin xyz="-0.2 -0.24 ${-WHEEL_RADIUS+0.0115+0.05}" rpy="${-M_PI/2} 0 0"/>
-    </joint>
-    <link name="caster_back_right_link">
-      <collision>
-        <geometry>
-          <cylinder length="0.06" radius="0.05"/>
-        </geometry>
-        <origin rpy="0 0 0" xyz="0 0 0.03"/>
-      </collision>
-      <inertial>
-        <mass value="0.0001" />
-        <origin xyz="0 0 0" />
-        <inertia
-        ixx="0.0069046"
-        ixy="-3.8717E-08"
-        ixz="2.0707E-07"
-        iyy="0.01"
-        iyz="-1.0124E-07"
-        izz="0.0069054" />
-      </inertial>
-      <damping>0.5</damping>
-    </link>
-<link
-    name="left_wheel_link">
-    <inertial>
-      <origin
-        xyz="9.16610941069373E-06 4.59070539915452E-09 8.0609835912647E-06"
-        rpy="0 0 0" />
-    <mass
-        value="1.5" />
-      <inertia
-        ixx="0.0069046"
-        ixy="-3.8717E-08"
-        ixz="2.0707E-07"
-        iyy="0.01"
-        iyz="-1.0124E-07"
-        izz="0.0069054" />
-      </inertial>
-    <visual>
-      <origin
-        xyz="0 0 0"
-        rpy="0 0 0" />
-      <geometry>
-        <mesh
-          filename="package://mobilican_description/armadillo_2/mesh/left_wheel_link.STL" />
-      </geometry>
-      <material
-        name="">
-        <color
-          rgba="0.792156862745098 0.819607843137255 0.933333333333333 1" />
-      </material>
-    </visual>
-    <collision>
-      <origin
-        xyz="0 0 0"
-        rpy="${M_PI/2} 0 0" />
-      <geometry>
-      <cylinder  length="0.07" radius="${WHEEL_RADIUS}"/>
-      </geometry>
-    </collision>
-    <damping>0.5</damping>
-  </link>
-  <joint
-    name="left_wheel_joint"
-    type="continuous">
-    <origin
-      xyz="0.063115 0.16085 0.0115"
-      rpy="0 0 0" />
-    <parent
-      link="base_link" />
-    <child
-      link="left_wheel_link" />
-    <axis
-      xyz="0 1 0" />
-    <limit
-      effort="0.1"
-      velocity="10.0" />
-  </joint>
- <link
-    name="right_wheel_link">
-    <inertial>
-      <origin
-        xyz="9.16610941069373E-06 -4.99540929455033E-06 8.06098359126817E-06"
-        rpy="0 0 0" />
-       <mass
-        value="1.5" />
-      <inertia
-        ixx="0.0069046"
-        ixy="-3.8717E-08"
-        ixz="-2.0707E-07"
-        iyy="0.01"
-        iyz="1.0124E-07"
-        izz="0.0069054" />
-    </inertial>
-    <visual>
-      <origin
-        xyz="0 0 0"
-        rpy="0 0 0" />
-      <geometry>
-        <mesh
-          filename="package://mobilican_description/armadillo_2/mesh/right_wheel_link.STL" />
-      </geometry>
-      <material
-        name="">
-        <color
-          rgba="0.792156862745098 0.819607843137255 0.933333333333333 1" />
-      </material>
-    </visual>
-   <collision>
-      <origin
-        xyz="0 0 0"
-        rpy="${M_PI/2} 0 0" />
-      <geometry>
-      <cylinder  length="0.07" radius="${WHEEL_RADIUS}"/>
-      </geometry>
-    </collision>
-    <damping>0.5</damping>
-  </link>
-  <joint
-    name="right_wheel_joint"
-    type="continuous">
-    <origin
-      xyz="0.063115 -0.16085 0.0115"
-      rpy="0 0 0" />
-    <parent
-      link="base_link" />
-    <child
-      link="right_wheel_link" />
-    <axis
-      xyz="0 1 0" />
-    <limit
-      effort="0.1"
-      velocity="10.0" />
-  </joint>
- <link
-    name="caster_left_link">
-     <inertial>
-      <origin
-        xyz="9.16610941069373E-06 -4.99540929455033E-06 8.06098359126817E-06"
-        rpy="0 0 0" />
-       <mass
-        value="20" />
-      <inertia
-        ixx="0.0069046"
-        ixy="-3.8717E-08"
-        ixz="-2.0707E-07"
-        iyy="0.01"
-        iyz="1.0124E-07"
-        izz="0.0069054" />
-    </inertial>
-    <visual>
-      <origin
-        xyz="0 0 0"
-        rpy="0 0 0" />
-      <geometry>
-        <mesh
-          filename="package://mobilican_description/armadillo_2/mesh/caster_left_link.STL" />
-      </geometry>
-      <material
-        name="">
-        <color
-          rgba="0.792156862745098 0.819607843137255 0.933333333333333 1" />
-      </material>
-    </visual>
-  </link>
-  <link
-    name="laser_link" />
-  <joint
-    name="laser_joint"
-    type="fixed">
-    <origin
-      xyz="0.20337 0 0.143"
-      rpy="0 0 0" />
-    <parent
-      link="base_link" />
-    <child
-      link="laser_link" />
-    <axis
-      xyz="0 0 0" />
-  </joint>
-  <link
-    name="front_urf_link" />
-  <joint
-    name="front_urf_joint"
-    type="fixed">
-    <origin
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