Commit message: fixed armadillo inertia and mass

File: mobilican_description/armadillo_2/urdf/armadillo2.xacro (robot description, xacro)
@@ -3,12 +3,12 @@
   <xacro:property name="M_PI" value="3.1415926535897931" />
   <xacro:property name="WHEEL_RADIUS" value="0.1016" />
-  <!-- <xacro:include filename="$(find mobilican_description)/armadillo_2/urdf/intel_d435.urdf"/>
-<link name="base_footprint"/>
- <joint name="base_footprint_joint" type="fixed">
+  <xacro:include filename="$(find mobilican_description)/armadillo_2/urdf/intel_d435.urdf"/>
+ <link name="base_footprint"/>
+<joint name="base_footprint_joint" type="fixed">
     <parent link="base_footprint"/>
     <child link="base_link"/>
     <origin xyz="0.00 0.00 ${WHEEL_RADIUS-0.0115}" rpy="0.0 0.0 0.0"/>
-  </joint>  -->
-  <!-- <link name="base_link">
+  </joint>
+  <link name="base_link">
     <inertial>
       <origin xyz=" -0.0456493 0.0002660 0.1875887" rpy="0 0 0" />
@@ -31,6 +31,6 @@
       </geometry>
     </collision>
-  </link> -->
-  <!-- <link name="left_wheel_link">
+  </link>
+<link name="left_wheel_link">
     <inertial>
       <origin xyz="9.16610941069373E-06 4.59070539915452E-09 8.0609835912647E-06" rpy="0 0 0" />
@@ -53,14 +53,14 @@
       </geometry>
     </collision>
-    <damping>0.5</damping>
-  </link> -->
-  <!-- <joint name="left_wheel_joint" type="continuous">
+    <!-- <damping>0.5</damping> -->
+  </link>
+  <joint name="left_wheel_joint" type="continuous">
     <origin xyz="0.063115 0.16085 0.0115" rpy="0 0 0" />
     <parent link="base_link" />
     <child link="left_wheel_link" />
     <axis xyz="0 1 0" />
-    <limit effort="0.1" velocity="10.0" />
-  </joint> -->
- <!-- <link name="right_wheel_link">
+    <limit effort="10.1" velocity="10.0" />
+  </joint>
+ <link name="right_wheel_link">
     <inertial>
       <origin xyz="9.16610941069373E-06 -4.99540929455033E-06 8.06098359126817E-06" rpy="0 0 0" />
@@ -83,17 +83,17 @@
       </geometry>
     </collision>
-    <damping>0.5</damping>
-  </link> -->
-  <!-- <joint name="right_wheel_joint" type="continuous">
+    <!-- <damping>0.5</damping> -->
+  </link>
+  <joint name="right_wheel_joint" type="continuous">
     <origin xyz="0.063115 -0.16085 0.0115" rpy="0 0 0" />
     <parent link="base_link" />
     <child link="right_wheel_link" />
     <axis xyz="0 1 0" />
-    <limit effort="0.1" velocity="10.0" />
-  </joint> -->
- <!-- <link name="caster_left_link">
+    <limit effort="10.1" velocity="10.0" />
+  </joint>
+ <link name="caster_left_link">
      <inertial>
       <origin
-        xyz="-0.2215584 0.1690000 -0.0478000"
+        xyz="0.0 0.0 0.0"
         rpy="0 0 0" />
        <mass
@@ -122,30 +122,39 @@
       </geometry>
     </collision>
-  </link> -->
-  <!-- <link name="laser_link" /> -->
-  <!-- <joint name="laser_joint" type="fixed">
+  </link>
+  <link name="laser_link" />
+  <joint name="laser_joint" type="fixed">
     <origin xyz="0.20337 0 0.143" rpy="0 0 0" />
     <parent link="base_link" />
     <child link="laser_link" />
     <axis xyz="0 0 0" />
-  </joint> -->
-  <!-- <link name="front_urf_link" /> -->
-  <!-- <joint name="front_urf_joint" type="fixed">
+  </joint>
+  <link name="front_urf_link" />
+  <joint name="front_urf_joint" type="fixed">
     <origin xyz="0.24229 0.00011161 0.068509" rpy="0 0 0" />
     <parent link="base_link" />
     <child link="front_urf_link" />
     <axis xyz="0 0 0" />
-  </joint> -->
-  <!-- <joint name="caster_left_joint" type="fixed">
+  </joint>
+  <joint name="caster_left_joint" type="fixed">
     <origin xyz="-0.221558374889189 0.168999999975415 -0.0596832588142329" rpy="0 0 0" />
     <parent link="base_link" />
     <child link="caster_left_link" />
     <axis xyz="0 0 0" />
-  </joint> -->
-  <!-- <link name="caster_right_link">
+  </joint>
+  <link name="caster_right_link">
       <inertial>
-      <origin xyz="9.16610941069373E-06 -4.99540929455033E-06 8.06098359126817E-06" rpy="0 0 0" />
-       <mass value="20" />
-      <inertia ixx="0.0069046" ixy="-3.8717E-08" ixz="-2.0707E-07" iyy="0.01" iyz="1.0124E-07" izz="0.0069054" />
+      <origin
+        xyz="0.0 0.0 0.0"
+        rpy="0 0 0" />
+       <mass
+        value="0.1" />
+      <inertia
+        ixx="0.0000224"
+        ixy="0.0000001"
+        ixz="0.0000006"
+        iyy="0.0000356"
+        iyz="0.0000001"
+        izz="0.0000211" />
     </inertial>
     <visual>
@@ -158,40 +167,66 @@
       </material>
     </visual>
-  </link> -->
-  <!-- <joint name="caster_right_joint" type="fixed">
+    <collision>
+      <origin xyz="0 0 0" rpy="1.57079632679 0 0" />
+      <geometry>
+      <cylinder length="0.018" radius="0.025"/>
+      </geometry>
+    </collision>
+  </link>
+  <joint name="caster_right_joint" type="fixed">
     <origin xyz="-0.221558374889189 -0.168999999975416 -0.0596832588142329" rpy="0 0 0" />
     <parent link="base_link" />
     <child link="caster_right_link" />
     <axis xyz="0 0 0" />
-  </joint> -->
-  <!-- <link name="torso_link">
+  </joint>
+<link
+    name="torso_link">
   <inertial>
-      <origin xyz="-0.059654 -0.000364 0.549359" rpy="0 0 0" />
-     <mass value="0.005" />
-      <inertia ixx="0.09579" ixy="2.4285E-05" ixz="-0.0045097" iyy="0.0001" iyz="-7.4938E-05" izz="0.00032852" />
-    </inertial>
-    <visual>
-      <origin xyz="0 0 0" rpy="0 0 0" />
-      <geometry>
-        <mesh filename="package://mobilican_description/armadillo_2/mesh/torso_link.STL" />
-      </geometry>
-      <material name="">
-        <color rgba="0.79216 0.81961 0.93333 1" />
+      <origin
+        xyz="-0.0624070 -0.0007353 0.5681605"
+        rpy="0 0 0" />
+     <mass
+        value="12.9807194" />
+      <inertia
+        ixx="0.8307393"
+        ixy="0.0004327"
+        ixz="-0.1085574"
+        iyy="0.7817095"
+        iyz="-0.0020591"
+        izz="0.2750408" />
+    </inertial>
+    <visual>
+      <origin
+        xyz="0 0 0"
+        rpy="0 0 0" />
+      <geometry>
+        <mesh
+          filename="package://mobilican_description/armadillo_2/mesh/torso_link.STL" />
+      </geometry>
+      <material
+        name="">
+        <color
+          rgba="0.79216 0.81961 0.93333 1" />
       </material>
     </visual>
     <collision name="torso">
-      <origin xyz="0 0 0" rpy="0 0 0" />
-      <geometry>
-        <mesh filename="package://mobilican_description/armadillo_2/mesh/torso_link.STL" />
+      <origin
+        xyz="0 0 0"
+        rpy="0 0 0" />
+      <geometry>
+        <mesh
+          filename="package://mobilican_description/armadillo_2/mesh/torso_link.STL" />
       </geometry>
     </collision>
      <collision name="safty box">
-      <origin xyz="0 -0.03 0.9" rpy="0 0 0" />
+      <origin
+        xyz="0 -0.03 0.9"
+        rpy="0 0 0" />
       <geometry>
         <box size="0.09 0.5 0.6"/>
       </geometry>
     </collision>
-  </link> -->
-  <!-- <joint name="torso_joint" type="prismatic">
+  </link>
+  <joint name="torso_joint" type="prismatic">
     <origin xyz="0 0 0" rpy="0 0 0" />
     <parent link="base_link" />
@@ -199,6 +234,6 @@
     <axis xyz="0 0 1" />
     <limit lower="0.05" upper="0.40" effort="0.001" velocity="0.1" />
-  </joint> -->
-  <!-- <link name="head_pan_link">
+  </joint>
+  <link name="head_pan_link">
   <inertial>
       <origin
@@ -230,6 +265,6 @@
       </geometry>
     </collision>
-  </link> -->
-  <!-- <joint name="head_pan_joint" type="revolute">
+  </link>
+  <joint name="head_pan_joint" type="revolute">
     <origin xyz="-0.055768 0 0.932" rpy="0 0 0" />
     <parent link="torso_link" />
@@ -237,6 +272,6 @@
     <axis xyz="0 0 1" />
     <limit upper="${3.1415926535897/4.0}" lower="${-3.1415926535897/4.0}" effort="0.5" velocity="2" />
-  </joint> -->
-  <!-- <link name="head_tilt_link">
+  </joint>
+  <link name="head_tilt_link">
     <inertial>
       <origin xyz="-0.002725 0.0002761 0.0027" rpy="0 0 0" />
@@ -259,6 +294,6 @@
       </geometry>
     </collision>
-  </link> -->
-  <!-- <joint name="head_tilt_joint" type="revolute">
+  </link>
+  <joint name="head_tilt_joint" type="revolute">
     <origin xyz="0 0 0.041" rpy="0 0 0" />
     <parent link="head_pan_link" />
@@ -266,59 +301,77 @@
     <axis xyz="0 1 0" />
     <limit upper="${50.0*M_PI/180.0}" lower="${-M_PI/6}" effort="0.5" velocity="2" />
-  </joint> -->
-  <!-- <link name="kinect2_link" /> -->
-  <!-- <joint name="kinect2_joint" type="fixed">
+  </joint>
+  <link name="kinect2_link" />
+  <joint name="kinect2_joint" type="fixed">
     <origin xyz="0.053 0.0073569 0.070961" rpy="0 0 0" />
     <parent link="head_tilt_link" />
     <child link="kinect2_link" />
     <axis xyz="0 0 0" />
-  </joint> -->
-   <!-- <joint name="kinect2_rgb_joint" type="fixed">
+  </joint>
+   <joint name="kinect2_rgb_joint" type="fixed">
       <origin xyz="0 -0.0935 0" rpy="0 0 0"/>
       <parent link="kinect2_link"/>
       <child link="kinect2_rgb_frame" />
-    </joint> -->
-    <!-- <link name="kinect2_rgb_frame"/> -->
-      <!-- <joint name="kinect2_rgb_optical_joint" type="fixed">
+    </joint>
+    <link name="kinect2_rgb_frame"/>
+      <joint name="kinect2_rgb_optical_joint" type="fixed">
 	<origin xyz="0 0 0" rpy="${-M_PI/2} 0 ${-M_PI/2}" />
 	<parent link="kinect2_rgb_frame" />
 	<child link="kinect2_rgb_optical_frame" />
-      </joint> -->
-      <!-- <link name="kinect2_rgb_optical_frame" /> -->
-	<!-- <joint name="kinect2_depth_joint" type="fixed">
+      </joint>
+      <link name="kinect2_rgb_optical_frame" />
+	<joint name="kinect2_depth_joint" type="fixed">
 	  <origin xyz="0 0 0" rpy="0 0 0" />
 	  <parent link="kinect2_rgb_frame" />
 	  <child link="kinect2_depth_frame" />
-	</joint> -->
-	<!-- <link name="kinect2_depth_frame" /> -->
-	  <!-- <joint name="kinect2_depth_optical_joint" type="fixed">
+	</joint>
+	<link name="kinect2_depth_frame" />
+	  <joint name="kinect2_depth_optical_joint" type="fixed">
 	    <origin xyz="0 0 0" rpy="${-M_PI/2} 0 ${-M_PI/2}" />
 	    <parent link="kinect2_depth_frame" />
 	    <child link="kinect2_depth_optical_frame" />
-	  </joint> -->
-	  <!-- <link name="kinect2_depth_optical_frame" /> -->
-  <!-- <link name="rotation1_link">
-    <inertial>
-      <origin xyz="-3.5316E-10 0.0073117 0.032399" rpy="0 0 0" />
-      <mass value="0.008" />
-      <inertia ixx="0.00055596" ixy="0.0" ixz="0.0" iyy="0.00016945" iyz="0.0" izz="0.00055286" />
-    </inertial>
-    <visual>
-      <origin xyz="0 0 0" rpy="0 0 0" />
-      <geometry>
-        <mesh filename="package://mobilican_description/armadillo_2/mesh/rotation1_link.STL" />
-      </geometry>
-      <material name="">
-        <color rgba="0.89804 0.91765 0.92941 1" />
-      </material>
-    </visual>
-    <collision>
-      <origin xyz="0 0 0" rpy="0 0 0" />
-      <geometry>
-        <mesh filename="package://mobilican_description/armadillo_2/mesh/rotation1_link.STL" />
-      </geometry>
-    </collision>
-  </link> -->
-  <!-- <joint name="rotation1_joint" type="revolute">
+	  </joint>
+	  <link name="kinect2_depth_optical_frame" />
+  <link
+    name="rotation1_link">
+    <inertial>
+      <origin
+        xyz="-1.0226405833258E-09 0.00201234378656519 0.0312057226305194"
+        rpy="0 0 0" />
+      <mass
+        value="0.402504348648636" />
+      <inertia
+        ixx="0.000224140297179524"
+        ixy="0.0"
+        ixz="0.0"
+        iyy="0.000224140297179524"
+        iyz="0.0"
+        izz="0.000201895164099562" />
+    </inertial>
+    <visual>
+      <origin
+        xyz="0 0 0"
+        rpy="0 0 0" />
+      <geometry>
+        <mesh
+          filename="package://mobilican_description/armadillo_2/mesh/rotation1_link.STL" />
+      </geometry>
+      <material
+        name="">
+        <color
+          rgba="0.89804 0.91765 0.92941 1" />
+      </material>
+    </visual>
+    <collision>
+      <origin
+        xyz="0 0 0"
+        rpy="0 0 0" />
+      <geometry>
+        <mesh
+          filename="package://mobilican_description/armadillo_2/mesh/rotation1_link.STL" />
+      </geometry>
+    </collision>
+  </link>
+  <joint name="rotation1_joint" type="revolute">
     <origin xyz="0.11617 0 0.3885" rpy="0 0 0" />
     <parent link="torso_link" />
@@ -326,28 +379,46 @@
     <axis xyz="0 0 1" />
        <limit effort="0.001" lower="-1.57" upper="1.57" velocity="2.0" />
-  </joint> -->
-  <!-- <link name="shoulder1_link">
-    <inertial>
-      <origin xyz="0.01628 -0.03243 0.20044" rpy="0 0 0" />
-      <mass value="0.009" />
-      <inertia ixx="0.0043595" ixy="0.0" ixz="0.00053636" iyy="0.0041046" iyz="0.0" izz="0.00081871" />
-    </inertial>
-    <visual>
-      <origin xyz="0 0 0" rpy="0 0 0" />
-      <geometry>
-        <mesh filename="package://mobilican_description/armadillo_2/mesh/shoulder1_link.STL" />
-      </geometry>
-      <material name="">
-        <color rgba="0.89804 0.91765 0.92941 1" />
-      </material>
-    </visual>
-    <collision>
-      <origin xyz="0 0 0" rpy="0 0 0" />
-      <geometry>
-        <mesh filename="package://mobilican_description/armadillo_2/mesh/shoulder1_link.STL" />
-      </geometry>
-    </collision>
-  </link> -->
-  <!-- <joint name="shoulder1_joint" type="revolute">
+  </joint>
+  <link
+    name="shoulder1_link">
+    <inertial>
+      <origin
+        xyz="0.0103824594991275 -0.0333360824774125 0.171916793222649"
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
File: mobilican_description/armadillo_2/urdf/intel_d435.urdf (robot description, URDF)
Before this commit: robot intel_d435, 9 links, 8 joints
Links:
- removed link camera_depth_frame
- removed link camera_depth_optical_frame
- removed link camera_fisheye_frame
- removed link camera_fisheye_optical_frame
- removed link camera_left_ir_frame
- removed link camera_left_ir_optical_frame
- removed link camera_right_ir_frame
- removed link camera_right_ir_optical_frame
Joints:
- removed joint camera_depth_joint
- removed joint camera_depth_optical_joint
- removed joint camera_fisheye_joint
- removed joint camera_fisheye_optical_joint
- removed joint camera_left_ir_joint
- removed joint camera_left_ir_optical_joint
- removed joint camera_right_ir_joint
- removed joint camera_right_ir_optical_joint

Commit message: arm pid gazebo

File: mobilican_description/armadillo_2/urdf/armadillo2.xacro (robot description, xacro)
@@ -60,5 +60,5 @@
     <child link="left_wheel_link" />
     <axis xyz="0 1 0" />
-    <limit effort="10.1" velocity="10.0" />
+    <limit effort="100" velocity="10.0" />
   </joint>
  <link name="right_wheel_link">
@@ -83,5 +83,4 @@
       </geometry>
     </collision>
-    <!-- <damping>0.5</damping> -->
   </link>
   <joint name="right_wheel_joint" type="continuous">
@@ -90,5 +89,5 @@
     <child link="right_wheel_link" />
     <axis xyz="0 1 0" />
-    <limit effort="10.1" velocity="10.0" />
+    <limit effort="100" velocity="10.0" />
   </joint>
  <link name="caster_left_link">
@@ -233,5 +232,5 @@
     <child link="torso_link" />
     <axis xyz="0 0 1" />
-    <limit lower="0.05" upper="0.40" effort="0.001" velocity="0.1" />
+    <limit lower="0.05" upper="0.40" effort="10" velocity="0.1" />
   </joint>
   <link name="head_pan_link">
@@ -271,5 +270,5 @@
     <child link="head_pan_link" />
     <axis xyz="0 0 1" />
-    <limit upper="${3.1415926535897/4.0}" lower="${-3.1415926535897/4.0}" effort="0.5" velocity="2" />
+    <limit upper="${3.1415926535897/4.0}" lower="${-3.1415926535897/4.0}" effort="10" velocity="2" />
   </joint>
   <link name="head_tilt_link">
@@ -300,5 +299,5 @@
     <child link="head_tilt_link" />
     <axis xyz="0 1 0" />
-    <limit upper="${50.0*M_PI/180.0}" lower="${-M_PI/6}" effort="0.5" velocity="2" />
+    <limit upper="${50.0*M_PI/180.0}" lower="${-M_PI/6}" effort="10" velocity="2" />
   </joint>
   <link name="kinect2_link" />
@@ -378,5 +377,5 @@
     <child link="rotation1_link" />
     <axis xyz="0 0 1" />
-       <limit effort="0.001" lower="-1.57" upper="1.57" velocity="2.0" />
+       <limit effort="50" lower="-1.57" upper="1.57" velocity="2.0" />
   </joint>
   <link
@@ -425,5 +424,5 @@
     <child link="shoulder1_link" />
     <axis xyz="0 1 0" />
-    <limit effort="0.01" lower="-1.57" upper="1.95" velocity="2.0" />
+    <limit effort="50" lower="-1.57" upper="1.95" velocity="2.0" />
   </joint>
 <link
@@ -472,5 +471,5 @@
     <child link="shoulder2_link" />
     <axis xyz="0 1 0" />
-    <limit effort="0.1" lower="-1.48" upper="2.3522" velocity="2.0" />
+    <limit effort="50" lower="-1.48" upper="2.3522" velocity="2.0" />
   </joint>
 <link
@@ -519,5 +518,5 @@
     <child link="rotation2_link" />
     <axis xyz="0 0 1" />
-   <limit effort="0.1" lower="-1.57" upper="1.57" velocity="2.0" />
+   <limit effort="40" lower="-1.57" upper="1.57" velocity="2.0" />
   </joint>
 <link
@@ -566,6 +565,6 @@
     <child link="shoulder3_link" />
     <axis xyz="0 1 0" />
-    <limit effort="0.1" lower="-1.57" upper="1.57" velocity="2.0" />
-    <dynamics damping="0.1"/>
+    <limit effort="40" lower="-1.57" upper="1.57" velocity="2.0" />
+    <!-- <dynamics damping="0.1"/>   -->
     </joint>
 <link
@@ -614,5 +613,5 @@
     <child link="wrist_link" />
     <axis xyz="0 1 0" />
- <limit effort="0.1" lower="-3.14" upper="3.14" velocity="2.0" />
+ <limit effort="30" lower="-3.14" upper="3.14" velocity="2.0" />
   </joint>
   <link name="gripper_link"/>
@@ -649,10 +648,10 @@
     <child link="left_finger_link" />
     <axis xyz="1 0 0" />
-    <limit effort="0.5" lower="-1.57" upper="1.57" velocity="0.1" />
-    <dynamics damping="0.1" friction="0.5"/>
+    <limit effort="5" lower="-1.57" upper="1.57" velocity="0.1" />
+    <!-- <dynamics damping="0.1" friction="0.5"/> -->
   </joint>
   <link name="right_finger_link">
      <inertial>
-      <origin xyz="5.5511E-17 0.015598 0.034754" rpy="0 0 0" />
+      <origin xyz="2.22044604925031E-16 -0.0155982142997538 0.0347541013107009" rpy="0 0 0" />
       <mass value="0.0172285040929193" />
       <inertia ixx="1.4683E-05" ixy="0.0" ixz="0.0" iyy="1.7304E-05" iyz="0.0" izz="4.5506E-06" />
@@ -661,5 +660,5 @@
       <origin xyz="0 0 0" rpy="0 0 0" />
       <geometry>
-        <mesh filename="package://mobilican_description/armadillo_2/mesh/left_finger_link.STL" />
+        <mesh filename="package://mobilican_description/armadillo_2/mesh/right_finger_link.STL" />
       </geometry>
       <material name="">
@@ -670,5 +669,5 @@
       <origin xyz="0 0 0" rpy="0 0 0" />
       <geometry>
-        <mesh filename="package://mobilican_description/armadillo_2/mesh/left_finger_link.STL" />
+        <mesh filename="package://mobilican_description/armadillo_2/mesh/right_finger_link.STL" />
       </geometry>
     </collision>
@@ -679,6 +678,6 @@
     <child link="right_finger_link" />
     <axis xyz="1 0 0" />
-  <limit effort="0.5" lower="-1.57" upper="1.57" velocity="0.1" />
-      <dynamics damping="0.1" friction="0.5"/>
+  <limit effort="5" lower="-1.57" upper="1.57" velocity="0.1" />
+      <!-- <dynamics damping="0.1" friction="0.5"/> -->
   </joint>
     <joint name="intel_d435_joint" type="fixed">

Commit message: added damping and friction to model

File: mobilican_description/armadillo_2/urdf/armadillo2.xacro (robot description, xacro)
@@ -271,4 +271,5 @@
     <axis xyz="0 0 1" />
     <limit upper="${3.1415926535897/4.0}" lower="${-3.1415926535897/4.0}" effort="10" velocity="2" />
+    <dynamics damping="0.7" friction="0.5"/>
   </joint>
   <link name="head_tilt_link">
@@ -300,4 +301,5 @@
     <axis xyz="0 1 0" />
     <limit upper="${50.0*M_PI/180.0}" lower="${-M_PI/6}" effort="10" velocity="2" />
+    <dynamics damping="0.7" friction="0.5"/>
   </joint>
   <link name="kinect2_link" />
@@ -378,4 +380,5 @@
     <axis xyz="0 0 1" />
        <limit effort="50" lower="-1.57" upper="1.57" velocity="2.0" />
+       <dynamics damping="0.7" friction="0.5"/>
   </joint>
   <link
@@ -425,4 +428,5 @@
     <axis xyz="0 1 0" />
     <limit effort="50" lower="-1.57" upper="1.95" velocity="2.0" />
+     <dynamics damping="0.7" friction="0.5"/>
   </joint>
 <link
@@ -472,4 +476,5 @@
     <axis xyz="0 1 0" />
     <limit effort="50" lower="-1.48" upper="2.3522" velocity="2.0" />
+    <dynamics damping="0.7" friction="0.5"/>
   </joint>
 <link
@@ -566,5 +571,5 @@
     <axis xyz="0 1 0" />
     <limit effort="40" lower="-1.57" upper="1.57" velocity="2.0" />
-    <!-- <dynamics damping="0.1"/>   -->
+    <dynamics damping="0.7" friction="0.5"/>
     </joint>
 <link
@@ -649,5 +654,5 @@
     <axis xyz="1 0 0" />
     <limit effort="5" lower="-1.57" upper="1.57" velocity="0.1" />
-    <!-- <dynamics damping="0.1" friction="0.5"/> -->
+    <dynamics damping="0.7" friction="0.5"/>
   </joint>
   <link name="right_finger_link">
@@ -679,5 +684,5 @@
     <axis xyz="1 0 0" />
   <limit effort="5" lower="-1.57" upper="1.57" velocity="0.1" />
-      <!-- <dynamics damping="0.1" friction="0.5"/> -->
+     <dynamics damping="0.7" friction="0.5"/>
   </joint>
     <joint name="intel_d435_joint" type="fixed">

Commit message: armadillo is stabilized driving fw and to the sides

File: mobilican_description/armadillo_2/urdf/armadillo2.xacro (robot description, xacro)
@@ -61,4 +61,5 @@
     <axis xyz="0 1 0" />
     <limit effort="100" velocity="10.0" />
+    <dynamics damping="0.7" friction="0.5"/>
   </joint>
  <link name="right_wheel_link">
@@ -90,4 +91,5 @@
     <axis xyz="0 1 0" />
     <limit effort="100" velocity="10.0" />
+    <dynamics damping="0.7" friction="0.5"/>
   </joint>
  <link name="caster_left_link">

File: mobilican_description/armadillo_2/urdf/armadillo2_gazebo.xacro (robot description, xacro)
@@ -149,22 +149,22 @@
     <gazebo reference="left_wheel_link">
         <!-- kp and kd for rubber -->
-        <kp>1000000.0</kp>
-        <kd>100.0</kd>
+        <kp>10000.0</kp>
+        <kd>10000.0</kd>
         <mu1>${mu1}</mu1>
         <mu2>${mu2}</mu2>
         <fdir1>1 0 0</fdir1>
         <maxVel>1.0</maxVel>
-        <minDepth>0.002</minDepth>
+        <minDepth>0.003</minDepth>
         <material>Gazebo/DarkGrey</material>
     </gazebo>
     <gazebo reference="right_wheel_link">
         <!-- kp and kd for rubber -->
-        <kp>1000000.0</kp>
-        <kd>100.0</kd>
+        <kp>10000.0</kp>
+        <kd>10000.0</kd>
         <mu1>${mu1}</mu1>
         <mu2>${mu2}</mu2>
         <fdir1>1 0 0</fdir1>
         <maxVel>1.0</maxVel>
-        <minDepth>0.002</minDepth>
+        <minDepth>0.003</minDepth>
         <material>Gazebo/DarkGrey</material>
     </gazebo>
