Commit message: stable realistic model for armadillo in gazebo :)

File: mobilican_description/armadillo_2/urdf/armadillo2.xacro (robot description, xacro)
@@ -99,11 +99,11 @@
         rpy="0 0 0" />
        <mass
-        value="0.1" />
+        value="10.1" />
       <inertia
         ixx="0.0000224"
-        ixy="0.0000001"
-        ixz="0.0000006"
+        ixy="0.0"
+        ixz="0.0"
         iyy="0.0000356"
-        iyz="0.0000001"
+        iyz="0.0"
         izz="0.0000211" />
     </inertial>
@@ -124,4 +124,47 @@
     </collision>
   </link>
+    <joint name="caster_left_joint" type="fixed">
+    <origin xyz="-0.221558374889189 0.168999999975415 -0.0596832588142329" rpy="0 0 0" />
+    <parent link="base_link" />
+    <child link="caster_left_link" />
+    <axis xyz="0 0 0" />
+  </joint>
+  <link name="caster_right_link">
+      <inertial>
+      <origin
+        xyz="0.0 0.0 0.0"
+        rpy="0 0 0" />
+       <mass
+        value="10.1" />
+      <inertia
+        ixx="0.0000224"
+        ixy="0.0"
+        ixz="0.0"
+        iyy="0.0000356"
+        iyz="0.0"
+        izz="0.0000211" />
+    </inertial>
+    <visual>
+      <origin xyz="0 0 0" rpy="0 0 0" />
+      <geometry>
+        <mesh filename="package://mobilican_description/armadillo_2/mesh/caster_right_link.STL" />
+      </geometry>
+      <material name="">
+        <color rgba="0.792156862745098 0.819607843137255 0.933333333333333 1" />
+      </material>
+    </visual>
+    <collision>
+      <origin xyz="0 0 0" rpy="1.57079632679 0 0" />
+      <geometry>
+      <cylinder length="0.018" radius="0.025"/>
+      </geometry>
+    </collision>
+  </link>
+  <joint name="caster_right_joint" type="fixed">
+    <origin xyz="-0.221558374889189 -0.168999999975416 -0.0596832588142329" rpy="0 0 0" />
+    <parent link="base_link" />
+    <child link="caster_right_link" />
+    <axis xyz="0 0 0" />
+  </joint>
   <link name="laser_link" />
   <joint name="laser_joint" type="fixed">
@@ -136,47 +179,4 @@
     <parent link="base_link" />
     <child link="front_urf_link" />
-    <axis xyz="0 0 0" />
-  </joint>
-  <joint name="caster_left_joint" type="fixed">
-    <origin xyz="-0.221558374889189 0.168999999975415 -0.0596832588142329" rpy="0 0 0" />
-    <parent link="base_link" />
-    <child link="caster_left_link" />
-    <axis xyz="0 0 0" />
-  </joint>
-  <link name="caster_right_link">
-      <inertial>
-      <origin
-        xyz="0.0 0.0 0.0"
-        rpy="0 0 0" />
-       <mass
-        value="0.1" />
-      <inertia
-        ixx="0.0000224"
-        ixy="0.0000001"
-        ixz="0.0000006"
-        iyy="0.0000356"
-        iyz="0.0000001"
-        izz="0.0000211" />
-    </inertial>
-    <visual>
-      <origin xyz="0 0 0" rpy="0 0 0" />
-      <geometry>
-        <mesh filename="package://mobilican_description/armadillo_2/mesh/caster_right_link.STL" />
-      </geometry>
-      <material name="">
-        <color rgba="0.792156862745098 0.819607843137255 0.933333333333333 1" />
-      </material>
-    </visual>
-    <collision>
-      <origin xyz="0 0 0" rpy="1.57079632679 0 0" />
-      <geometry>
-      <cylinder length="0.018" radius="0.025"/>
-      </geometry>
-    </collision>
-  </link>
-  <joint name="caster_right_joint" type="fixed">
-    <origin xyz="-0.221558374889189 -0.168999999975416 -0.0596832588142329" rpy="0 0 0" />
-    <parent link="base_link" />
-    <child link="caster_right_link" />
     <axis xyz="0 0 0" />
   </joint>

File: mobilican_description/armadillo_2/urdf/armadillo2_gazebo.xacro (robot description, xacro)
@@ -149,28 +149,28 @@
     <gazebo reference="left_wheel_link">
         <!-- kp and kd for rubber -->
-        <kp>10000.0</kp>
-        <kd>10000.0</kd>
+        <kp>1000000.0</kp>
+        <kd>100.0</kd>
         <mu1>${mu1}</mu1>
         <mu2>${mu2}</mu2>
         <fdir1>1 0 0</fdir1>
         <maxVel>1.0</maxVel>
-        <minDepth>0.003</minDepth>
+        <minDepth>0.001</minDepth>
         <material>Gazebo/DarkGrey</material>
     </gazebo>
     <gazebo reference="right_wheel_link">
         <!-- kp and kd for rubber -->
-        <kp>10000.0</kp>
-        <kd>10000.0</kd>
+        <kp>1000000.0</kp>
+        <kd>100.0</kd>
         <mu1>${mu1}</mu1>
         <mu2>${mu2}</mu2>
         <fdir1>1 0 0</fdir1>
         <maxVel>1.0</maxVel>
-        <minDepth>0.003</minDepth>
+        <minDepth>0.001</minDepth>
         <material>Gazebo/DarkGrey</material>
     </gazebo>
-    <gazebo reference="caster_back_left_link">
+    <gazebo reference="caster_left_link">
         <!-- kp and kd for rubber -->
         <kp>1000000.0</kp>
-        <kd>100.0</kd>
+        <kd>1000.0</kd>
         <mu1>0.0</mu1>
         <mu2>0.0</mu2>
@@ -180,8 +180,8 @@
         <material>Gazebo/DarkGrey</material>
     </gazebo>
-    <gazebo reference="caster_back_right_link">
+    <gazebo reference="caster_right_link">
     <!-- kp and kd for rubber -->
         <kp>1000000.0</kp>
-        <kd>100.0</kd>
+        <kd>1000.0</kd>
         <mu1>0.0</mu1>
         <mu2>0.0</mu2>
