Commit message: adapting all robots launch to generic mobilican launch

File: mobilican_description/armadillo2/urdf/armadillo2.xacro (robot description, xacro)
@@ -3,5 +3,5 @@
   <xacro:property name="M_PI" value="3.1415926535897931" />
   <xacro:property name="WHEEL_RADIUS" value="0.1016" />
-  <xacro:include filename="$(find mobilican_description)/armadillo_2/urdf/intel_d435.urdf"/>
+  <xacro:include filename="$(find mobilican_description)/armadillo2/urdf/intel_d435.urdf"/>
  <link name="base_footprint"/>
 <joint name="base_footprint_joint" type="fixed">
@@ -19,5 +19,5 @@
       <origin xyz="0 0 0" rpy="0 0 0" />
       <geometry>
-        <mesh filename="package://mobilican_description/armadillo_2/mesh/base_link.STL" />
+        <mesh filename="package://mobilican_description/armadillo2/mesh/base_link.STL" />
       </geometry>
       <material name="">
@@ -28,5 +28,5 @@
       <origin xyz="0 0 0" rpy="0 0 0" />
       <geometry>
-        <mesh filename="package://mobilican_description/armadillo_2/mesh/base_link.STL" />
+        <mesh filename="package://mobilican_description/armadillo2/mesh/base_link.STL" />
       </geometry>
     </collision>
@@ -41,5 +41,5 @@
       <origin xyz="0 0 0" rpy="0 0 0" />
       <geometry>
-        <mesh filename="package://mobilican_description/armadillo_2/mesh/left_wheel_link.STL" />
+        <mesh filename="package://mobilican_description/armadillo2/mesh/left_wheel_link.STL" />
       </geometry>
       <material name="">
@@ -72,5 +72,5 @@
       <origin xyz="0 0 0" rpy="0 0 0" />
       <geometry>
-        <mesh filename="package://mobilican_description/armadillo_2/mesh/right_wheel_link.STL" />
+        <mesh filename="package://mobilican_description/armadillo2/mesh/right_wheel_link.STL" />
       </geometry>
       <material name="">
@@ -111,5 +111,5 @@
       <origin xyz="0 0 0" rpy="0 0 0" />
       <geometry>
-        <mesh filename="package://mobilican_description/armadillo_2/mesh/caster_left_link.STL" />
+        <mesh filename="package://mobilican_description/armadillo2/mesh/caster_left_link.STL" />
       </geometry>
       <material name="">
@@ -148,5 +148,5 @@
       <origin xyz="0 0 0" rpy="0 0 0" />
       <geometry>
-        <mesh filename="package://mobilican_description/armadillo_2/mesh/caster_right_link.STL" />
+        <mesh filename="package://mobilican_description/armadillo2/mesh/caster_right_link.STL" />
       </geometry>
       <material name="">
@@ -203,5 +203,5 @@
       <geometry>
         <mesh
-          filename="package://mobilican_description/armadillo_2/mesh/torso_link.STL" />
+          filename="package://mobilican_description/armadillo2/mesh/torso_link.STL" />
       </geometry>
       <material
@@ -217,5 +217,5 @@
       <geometry>
         <mesh
-          filename="package://mobilican_description/armadillo_2/mesh/torso_link.STL" />
+          filename="package://mobilican_description/armadillo2/mesh/torso_link.STL" />
       </geometry>
     </collision>
@@ -254,5 +254,5 @@
       <origin xyz="0 0 0" rpy="0 0 0" />
       <geometry>
-        <mesh filename="package://mobilican_description/armadillo_2/mesh/head_pan_link.STL" />
+        <mesh filename="package://mobilican_description/armadillo2/mesh/head_pan_link.STL" />
       </geometry>
       <material name="">
@@ -263,5 +263,5 @@
       <origin xyz="0 0 0" rpy="0 0 0" />
       <geometry>
-        <mesh filename="package://mobilican_description/armadillo_2/mesh/head_pan_link.STL" />
+        <mesh filename="package://mobilican_description/armadillo2/mesh/head_pan_link.STL" />
       </geometry>
     </collision>
@@ -284,5 +284,5 @@
       <origin xyz="0 0 0" rpy="0 0 0" />
       <geometry>
-        <mesh filename="package://mobilican_description/armadillo_2/mesh/head_tilt_link.STL" />
+        <mesh filename="package://mobilican_description/armadillo2/mesh/head_tilt_link.STL" />
       </geometry>
       <material name="">
@@ -293,5 +293,5 @@
       <origin xyz="0 0 0" rpy="0 0 0" />
       <geometry>
-        <mesh filename="package://mobilican_description/armadillo_2/mesh/head_tilt_link.STL" />
+        <mesh filename="package://mobilican_description/armadillo2/mesh/head_tilt_link.STL" />
       </geometry>
     </collision>
@@ -358,5 +358,5 @@
       <geometry>
         <mesh
-          filename="package://mobilican_description/armadillo_2/mesh/rotation1_link.STL" />
+          filename="package://mobilican_description/armadillo2/mesh/rotation1_link.STL" />
       </geometry>
       <material
@@ -372,5 +372,5 @@
       <geometry>
         <mesh
-          filename="package://mobilican_description/armadillo_2/mesh/rotation1_link.STL" />
+          filename="package://mobilican_description/armadillo2/mesh/rotation1_link.STL" />
       </geometry>
     </collision>
@@ -406,5 +406,5 @@
       <geometry>
         <mesh
-          filename="package://mobilican_description/armadillo_2/mesh/shoulder1_link.STL" />
+          filename="package://mobilican_description/armadillo2/mesh/shoulder1_link.STL" />
       </geometry>
       <material
@@ -420,5 +420,5 @@
       <geometry>
         <mesh
-          filename="package://mobilican_description/armadillo_2/mesh/shoulder1_link.STL" />
+          filename="package://mobilican_description/armadillo2/mesh/shoulder1_link.STL" />
       </geometry>
     </collision>
@@ -454,5 +454,5 @@
       <geometry>
         <mesh
-          filename="package://mobilican_description/armadillo_2/mesh/shoulder2_link.STL" />
+          filename="package://mobilican_description/armadillo2/mesh/shoulder2_link.STL" />
       </geometry>
       <material
@@ -468,5 +468,5 @@
       <geometry>
         <mesh
-          filename="package://mobilican_description/armadillo_2/mesh/shoulder2_link.STL" />
+          filename="package://mobilican_description/armadillo2/mesh/shoulder2_link.STL" />
       </geometry>
     </collision>
@@ -502,5 +502,5 @@
       <geometry>
         <mesh
-          filename="package://mobilican_description/armadillo_2/mesh/rotation2_link.STL" />
+          filename="package://mobilican_description/armadillo2/mesh/rotation2_link.STL" />
       </geometry>
       <material
@@ -516,5 +516,5 @@
       <geometry>
         <mesh
-          filename="package://mobilican_description/armadillo_2/mesh/rotation2_link.STL" />
+          filename="package://mobilican_description/armadillo2/mesh/rotation2_link.STL" />
       </geometry>
     </collision>
@@ -549,5 +549,5 @@
       <geometry>
         <mesh
-          filename="package://mobilican_description/armadillo_2/mesh/shoulder3_link.STL" />
+          filename="package://mobilican_description/armadillo2/mesh/shoulder3_link.STL" />
       </geometry>
       <material
@@ -563,5 +563,5 @@
       <geometry>
         <mesh
-          filename="package://mobilican_description/armadillo_2/mesh/shoulder3_link.STL" />
+          filename="package://mobilican_description/armadillo2/mesh/shoulder3_link.STL" />
       </geometry>
     </collision>
@@ -597,5 +597,5 @@
       <geometry>
         <mesh
-          filename="package://mobilican_description/armadillo_2/mesh/wrist_link.STL" />
+          filename="package://mobilican_description/armadillo2/mesh/wrist_link.STL" />
       </geometry>
       <material
@@ -611,5 +611,5 @@
       <geometry>
         <mesh
-          filename="package://mobilican_description/armadillo_2/mesh/wrist_link.STL" />
+          filename="package://mobilican_description/armadillo2/mesh/wrist_link.STL" />
       </geometry>
     </collision>
@@ -637,5 +637,5 @@
       <origin xyz="0 0 0" rpy="0 0 0" />
       <geometry>
-        <mesh filename="package://mobilican_description/armadillo_2/mesh/left_finger_link.STL" />
+        <mesh filename="package://mobilican_description/armadillo2/mesh/left_finger_link.STL" />
       </geometry>
       <material name="">
@@ -646,5 +646,5 @@
       <origin xyz="0 0 0" rpy="0 0 0" />
       <geometry>
-        <mesh filename="package://mobilican_description/armadillo_2/mesh/left_finger_link.STL" />
+        <mesh filename="package://mobilican_description/armadillo2/mesh/left_finger_link.STL" />
       </geometry>
     </collision>
@@ -667,5 +667,5 @@
       <origin xyz="0 0 0" rpy="0 0 0" />
       <geometry>
-        <mesh filename="package://mobilican_description/armadillo_2/mesh/right_finger_link.STL" />
+        <mesh filename="package://mobilican_description/armadillo2/mesh/right_finger_link.STL" />
       </geometry>
       <material name="">
@@ -676,5 +676,5 @@
       <origin xyz="0 0 0" rpy="0 0 0" />
       <geometry>
-        <mesh filename="package://mobilican_description/armadillo_2/mesh/right_finger_link.STL" />
+        <mesh filename="package://mobilican_description/armadillo2/mesh/right_finger_link.STL" />
       </geometry>
     </collision>

File: mobilican_description/armadillo2/urdf/armadillo2_gazebo.xacro (robot description, xacro)
@@ -1,5 +1,5 @@
 <?xml version="1.0"?>
 <robot xmlns:xacro="http://www.ros.org/wiki/xacro" name="armadillo_robot" description="armadillo robot">
-    <xacro:include filename="$(find mobilican_description)/armadillo_2/urdf/armadillo2.xacro" />
+    <xacro:include filename="$(find mobilican_description)/armadillo2/urdf/armadillo2.xacro" />
     <xacro:arg name="kinect2" default="true"/>
     <xacro:arg name="kinect2_hz" default="30.0"/>

File: mobilican_description/armadillo2/urdf/intel_d435.urdf (robot description, URDF)
Before this commit: robot intel_d435, 9 links, 8 joints
Links:
- link camera_link: geometry collision mesh filename=package://mobilican_description/armadillo2/mesh/intel_d435.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; visual mesh filename=package://mobilican_description/armadillo2/mesh/intel_d435.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

File: mobilican_description/lizi2/urdf/lizi2.xacro (robot description, xacro)
@@ -25,5 +25,5 @@
       <geometry>
         <mesh
-          filename="package://mobilican_description/lizi_2/meshes/base.STL" />
+          filename="package://mobilican_description/lizi2/meshes/base.STL" />
       </geometry>
       <material
@@ -39,5 +39,5 @@
       <geometry>
         <mesh
-          filename="package://mobilican_description/lizi_2/meshes/base.STL" />
+          filename="package://mobilican_description/lizi2/meshes/base.STL" />
       </geometry>
     </collision>
@@ -80,5 +80,5 @@
       <geometry>
         <mesh
-          filename="package://mobilican_description/lizi_2/meshes/lidar.STL" />
+          filename="package://mobilican_description/lizi2/meshes/lidar.STL" />
       </geometry>
       <material
@@ -94,5 +94,5 @@
       <geometry>
         <mesh
-          filename="package://mobilican_description/lizi_2/meshes/lidar.STL" />
+          filename="package://mobilican_description/lizi2/meshes/lidar.STL" />
       </geometry>
     </collision>
@@ -133,5 +133,5 @@
       <geometry>
         <mesh
-          filename="package://mobilican_description/lizi_2/meshes/depth_cam.STL" />
+          filename="package://mobilican_description/lizi2/meshes/depth_cam.STL" />
       </geometry>
       <material
@@ -147,5 +147,5 @@
       <geometry>
         <mesh
-          filename="package://mobilican_description/lizi_2/meshes/depth_cam.STL" />
+          filename="package://mobilican_description/lizi2/meshes/depth_cam.STL" />
       </geometry>
     </collision>
@@ -231,5 +231,5 @@
       <geometry>
         <mesh
-          filename="package://mobilican_description/lizi_2/meshes/wheel.STL" />
+          filename="package://mobilican_description/lizi2/meshes/wheel.STL" />
       </geometry>
       <material
@@ -283,5 +283,5 @@
       <geometry>
         <mesh
-          filename="package://mobilican_description/lizi_2/meshes/wheel.STL" />
+          filename="package://mobilican_description/lizi2/meshes/wheel.STL" />
       </geometry>
       <material
@@ -335,5 +335,5 @@
       <geometry>
         <mesh
-          filename="package://mobilican_description/lizi_2/meshes/wheel.STL" />
+          filename="package://mobilican_description/lizi2/meshes/wheel.STL" />
       </geometry>
       <material
@@ -387,5 +387,5 @@
       <geometry>
         <mesh
-          filename="package://mobilican_description/lizi_2/meshes/wheel.STL" />
+          filename="package://mobilican_description/lizi2/meshes/wheel.STL" />
       </geometry>
       <material

File: mobilican_description/lizi2/urdf/lizi2_gazebo.xacro (robot description, xacro)
@@ -1,5 +1,5 @@
 <?xml version="1.0"?>
 <robot xmlns:xacro="http://www.ros.org/wiki/xacro" name="lizi" description="Lizi robot">
-    <xacro:include filename="$(find mobilican_description)/lizi_2/urdf/lizi.xacro" />
+    <xacro:include filename="$(find mobilican_description)/lizi2/urdf/lizi2.xacro" />
     <xacro:include filename="$(find mobilican_gazebo)/macros/depth_cam.xacro" />
     <xacro:include filename="$(find mobilican_gazebo)/macros/cam.xacro" />
@@ -11,10 +11,10 @@
     <xacro:property name="URF_FOV" value="${10.0*M_PI/180}" />
     <xacro:arg name="controllers" default="true"/>
-    <xacro:arg name="urf" default="false"/>
-    <xacro:arg name="imu" default="false"/>
-    <xacro:arg name="gps" default="false"/>
-    <xacro:arg name="lidar" default="false"/>
-    <xacro:arg name="cam" default="false"/>
-    <xacro:arg name="depth_cam" default="false"/>
+    <xacro:arg name="urf" default="true"/>
+    <xacro:arg name="imu" default="true"/>
+    <xacro:arg name="gps" default="true"/>
+    <xacro:arg name="lidar" default="true"/>
+    <xacro:arg name="cam" default="true"/>
+    <xacro:arg name="depth_cam" default="true"/>
    <xacro:if value="$(arg cam)">
         <xacro:Camera name="rgb_cam"
